File: Projects/ATTINY85/Chainable_RGB_LEDS/LED_Board.brd (EAGLE design)
At the start: 31 x 31 mm, 5 parts

Commit message: v1.0 Connector Board Completed
Parts:
- added E$1: (no value), con-molex:7395-04
- moved E$5 7.62 mm to (20.3, 27.9)
Connections:
- net S$1: now also E$1.2
- net S$2: now also E$1.4, E$6.3; no longer E$2.1
- net S$4: now also E$1.3, E$2.1; no longer E$6.3
- net S$8: now also E$1.1
Routing:
- net S$4: track 8.13 -> 21.4 mm
- net S$8: track 32.9 -> 40.5 mm
- net S$1: track 23.7 -> 31.3 mm
Changed lines of the file:
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@@
 <layer number="19" name="Unrouted" color="6" fill="1" visible="yes" active="yes"/>
 <layer number="20" name="Dimension" color="15" fill="1" visible="yes" active="yes"/>
-<layer number="21" name="tPlace" color="7" fill="1" visible="no" active="yes"/>
-<layer number="22" name="bPlace" color="7" fill="1" visible="no" active="yes"/>
-<layer number="23" name="tOrigins" color="15" fill="1" visible="no" active="yes"/>
-<layer number="24" name="bOrigins" color="15" fill="1" visible="no" active="yes"/>
-<layer number="25" name="tNames" color="7" fill="1" visible="no" active="yes"/>
-<layer number="26" name="bNames" color="7" fill="1" visible="no" active="yes"/>
-<layer number="27" name="tValues" color="7" fill="1" visible="no" active="yes"/>
-<layer number="28" name="bValues" color="7" fill="1" visible="no" active="yes"/>
+<layer number="21" name="tPlace" color="7" fill="1" visible="yes" active="yes"/>
+<layer number="22" name="bPlace" color="7" fill="1" visible="yes" active="yes"/>
+<layer number="23" name="tOrigins" color="15" fill="1" visible="yes" active="yes"/>
+<layer number="24" name="bOrigins" color="15" fill="1" visible="yes" active="yes"/>
+<layer number="25" name="tNames" color="7" fill="1" visible="yes" active="yes"/>
+<layer number="26" name="bNames" color="7" fill="1" visible="yes" active="yes"/>
+<layer number="27" name="tValues" color="7" fill="1" visible="yes" active="yes"/>
+<layer number="28" name="bValues" color="7" fill="1" visible="yes" active="yes"/>
 <layer number="29" name="tStop" color="7" fill="3" visible="no" active="yes"/>
 <layer number="30" name="bStop" color="7" fill="6" visible="no" active="yes"/>
@@
 <layer number="43" name="vRestrict" color="2" fill="10" visible="no" active="yes"/>
 <layer number="44" name="Drills" color="7" fill="1" visible="no" active="yes"/>
-<layer number="45" name="Holes" color="7" fill="1" visible="no" active="yes"/>
+<layer number="45" name="Holes" color="7" fill="1" visible="yes" active="yes"/>
 <layer number="46" name="Milling" color="3" fill="1" visible="no" active="yes"/>
 <layer number="47" name="Measures" color="7" fill="1" visible="no" active="yes"/>
@@
 <element name="E$3" library="resistor" package="0207/10" value="" x="24.13" y="11.43" rot="R180"/>
 <element name="E$4" library="resistor" package="0207/10" value="" x="24.13" y="7.62" rot="R180"/>
-<element name="E$5" library="con-molex" package="7395-04" value="" x="27.94" y="27.94" rot="R270"/>
 <element name="E$6" library="pinhead" package="1X04" value="" x="24.13" y="20.32"/>
+<element name="E$1" library="con-molex" package="7395-04" value="" x="27.94" y="27.94" rot="R90"/>
+<element name="E$5" library="con-molex" package="7395-04" value="" x="20.32" y="27.94" rot="R270"/>
 </elements>
 <signals>
 <signal name="S$3">
-</signal>
-<signal name="S$4">
-<contactref element="E$5" pad="2"/>
-<wire x1="27.94" y1="26.67" x2="26.8015125" y2="26.67" width="0.4064" layer="16"/>
-<wire x1="26.8015125" y1="26.67" x2="26.57700625" y2="26.57700625" width="0.4064" layer="16" curve="45"/>
-<wire x1="26.57700625" y1="26.57700625" x2="25.4" y2="25.4" width="0.4064" layer="16"/>
-<contactref element="E$6" pad="3"/>
-<wire x1="25.4" y1="25.4" x2="25.4" y2="20.32" width="0.4064" layer="16"/>
 </signal>
 <signal name="S$5">
@@
 <wire x1="30.57299375" y1="7.71299375" x2="35.56" y2="12.7" width="0.4064" layer="16"/>
 <wire x1="35.56" y1="12.7" x2="35.56" y2="27.94" width="0.4064" layer="16"/>
+<wire x1="35.56" y1="27.94" x2="31.75" y2="31.75" width="0.4064" layer="16"/>
+<contactref element="E$1" pad="1"/>
+<wire x1="27.94" y1="31.75" x2="31.75" y2="31.75" width="0.4064" layer="16"/>
 <contactref element="E$5" pad="4"/>
-<wire x1="27.94" y1="31.75" x2="31.75" y2="31.75" width="0.4064" layer="16"/>
-<wire x1="35.56" y1="27.94" x2="31.75" y2="31.75" width="0.4064" layer="16"/>
+<wire x1="20.32" y1="31.75" x2="27.94" y2="31.75" width="0.4064" layer="16"/>
 </signal>
 <signal name="S$1">
@@
 <wire x1="33.02" y1="13.97" x2="33.02" y2="26.67" width="0.4064" layer="16"/>
 <wire x1="33.02" y1="26.67" x2="30.48" y2="29.21" width="0.4064" layer="16"/>
+<contactref element="E$1" pad="2"/>
+<wire x1="30.48" y1="29.21" x2="27.94" y2="29.21" width="0.4064" layer="16"/>
 <contactref element="E$5" pad="3"/>
-<wire x1="30.48" y1="29.21" x2="27.94" y2="29.21" width="0.4064" layer="16"/>
+<wire x1="27.94" y1="29.21" x2="20.32" y2="29.21" width="0.4064" layer="16"/>
+</signal>
+<signal name="S$4">
+<contactref element="E$1" pad="3"/>
+<wire x1="27.94" y1="26.67" x2="29.21" y2="26.67" width="0.4064" layer="16"/>
+<wire x1="29.21" y1="26.67" x2="30.48" y2="25.4" width="0.4064" layer="16"/>
+<wire x1="30.48" y1="25.4" x2="30.48" y2="16.51" width="0.4064" layer="16"/>
+<contactref element="E$2" pad="1"/>
+<wire x1="30.48" y1="16.51" x2="29.21" y2="15.24" width="0.4064" layer="16"/>
+<contactref element="E$5" pad="2"/>
+<wire x1="20.32" y1="26.67" x2="27.94" y2="26.67" width="0.4064" layer="16"/>
 </signal>
 <signal name="S$2">
 <contactref element="E$5" pad="1"/>
-<wire x1="27.94" y1="24.13" x2="29.21" y2="24.13" width="0.4064" layer="16"/>
-<wire x1="29.21" y1="24.13" x2="30.48" y2="22.86" width="0.4064" layer="16"/>
-<wire x1="30.48" y1="22.86" x2="30.48" y2="16.51" width="0.4064" layer="16"/>
-<contactref element="E$2" pad="1"/>
-<wire x1="30.48" y1="16.51" x2="29.21" y2="15.24" width="0.4064" layer="16"/>
+<contactref element="E$1" pad="4"/>
+<wire x1="20.32" y1="24.13" x2="25.4" y2="24.13" width="0.4064" layer="16"/>
+<wire x1="27.94" y1="24.13" x2="25.4" y2="24.13" width="0.4064" layer="16"/>
+<contactref element="E$6" pad="3"/>
+<wire x1="25.4" y1="24.13" x2="25.4" y2="20.32" width="0.4064" layer="16"/>
 </signal>
 </signals>
